Commit message: minor changes

File: urdf/faro.xacro (robot description, xacro)
@@ -58,5 +58,5 @@
         <origin xyz="0.005 -0.072 -0.0234" rpy="0 0 0"/>
         <geometry>
-          <mesh filename="package://urdf_simple_description/meshes/wheel_1.stl" scale="0.001 0.001 0.001"/>
+          <mesh filename="package://faro_description/meshes/wheel_1.stl" scale="0.001 0.001 0.001"/>
         </geometry>
         <material name="silver"/>
@@ -65,5 +65,5 @@
         <origin xyz="0.005 -0.072 -0.0234" rpy="0 0 0"/>
         <geometry>
-          <mesh filename="package://urdf_simple_description/meshes/wheel_1.stl" scale="0.001 0.001 0.001"/>
+          <mesh filename="package://faro_description/meshes/wheel_1.stl" scale="0.001 0.001 0.001"/>
         </geometry>
       </collision>
@@ -92,5 +92,5 @@
         <origin xyz="0.005 0.072 -0.0234" rpy="0 0 0"/>
         <geometry>
-          <mesh filename="package://urdf_simple_description/meshes/wheel_2.stl" scale="0.001 0.001 0.001"/>
+          <mesh filename="package://faro_description/meshes/wheel_2.stl" scale="0.001 0.001 0.001"/>
         </geometry>
         <material name="silver"/>
@@ -99,5 +99,5 @@
         <origin xyz="0.005 0.072 -0.0234" rpy="0 0 0"/>
         <geometry>
-          <mesh filename="package://urdf_simple_description/meshes/wheel_2.stl" scale="0.001 0.001 0.001"/>
+          <mesh filename="package://faro_description/meshes/wheel_2.stl" scale="0.001 0.001 0.001"/>
         </geometry>
       </collision>

Commit message: new version urdf

File: urdf/faro.xacro (robot description, xacro)
@@ -7,179 +7,219 @@
   <joint name="dummy_joint" type="fixed">
       <parent link="dummy" />
-      <child link="Base1_link" />
-  </joint>
-  <link name="Base1_link">
-    <inertial>
-      <origin
-        xyz="5.1713E-10 -7.3629E-10 -8.9432E-11"
-        rpy="0 0 0" />
-      <mass
-        value="0.57317" />
-      <inertia
-        ixx="0.00079912"
-        ixy="1.6466E-06"
-        ixz="1.5171E-07"
-        iyy="0.0022607"
-        iyz="-9.1778E-09"
-        izz="0.0015696" />
-    </inertial>
-    <visual>
-      <origin
-        xyz="0 0 0"
-        rpy="0 0 0" />
-      <geometry>
-        <mesh
-          filename="package://faro_description/meshes/Base1_link.STL" />
-      </geometry>
-      <material
-        name="">
-        <color
-          rgba="0.79216 0.81961 0.93333 1" />
-      </material>
-    </visual>
-    <collision>
-      <origin
-        xyz="0 0 0"
-        rpy="0 0 0" />
-      <geometry>
-        <mesh
-          filename="package://faro_description/meshes/Base1_link.STL" />
-      </geometry>
-    </collision>
-  </link>
+      <child link="base_link" />
+  </joint>
+  <link
+    name="base_link">
+    <inertial>
+      <origin
+        xyz="0.00873430427479388 -0.00175292065981603 -1.60683999922646E-05"
+        rpy="0 0 0" />
+      <mass
+        value="0.451148910388453" />
+      <inertia
+        ixx="0.000741612731246182"
+        ixy="1.64659716773886E-06"
+        ixz="1.51707793234015E-07"
+        iyy="0.00220273812328352"
+        iyz="-9.17558592682493E-09"
+        izz="0.00147205616680342" />
+    </inertial>
+    <visual>
+      <origin
+        xyz="0 0 0"
+        rpy="0 0 0" />
+      <geometry>
+        <mesh
+          filename="package://faro_description/meshes/base_link.STL" />
+      </geometry>
+      <material
+        name="">
+        <color
+          rgba="0.498039215686275 0.498039215686275 0.498039215686275 1" />
+      </material>
+    </visual>
+    <collision>
+      <origin
+        xyz="0 0 0"
+        rpy="0 0 0" />
+      <geometry>
+        <mesh
+          filename="package://faro_description/meshes/base_link.STL" />
+      </geometry>
+    </collision>
+  </link>
+  <link
+    name="RodaEsferica_Link">
+    <inertial>
+      <origin
+        xyz="0.068659 -0.017264 0.00018379"
+        rpy="0 0 0" />
+      <mass
+        value="0.020844" />
+      <inertia
+        ixx="9.8497E-07"
+        ixy="1.4029E-22"
+        ixz="-7.8188E-23"
+        iyy="1.4E-06"
+        iyz="1.592E-22"
+        izz="8.9118E-07" />
+    </inertial>
+    <visual>
+      <origin
+        xyz="0 0 0"
+        rpy="0 0 0" />
+      <geometry>
+        <mesh
+          filename="package://faro_description/meshes/RodaEsferica_Link.STL" />
+      </geometry>
+      <material
+        name="">
+        <color
+          rgba="0.89804 0.89804 0.89804 1" />
+      </material>
+    </visual>
+    <collision>
+      <origin
+        xyz="0 0 0"
+        rpy="0 0 0" />
+      <geometry>
+        <mesh
+          filename="package://faro_description/meshes/RodaEsferica_Link.STL" />
+      </geometry>
+    </collision>
+  </link>
+  <joint
+    name="RodaEsferica_Joint"
+    type="fixed">
+    <origin
+      xyz="0 0 0"
+      rpy="1.5708 0 0" />
+    <parent
+      link="base_link" />
+    <child
+      link="RodaEsferica_Link" />
+    <axis
+      xyz="0 0 0" />
+    <dynamics
+      friction="0" />
+  </joint>
   <link
     name="RodaEsquerda_Link">
-      <inertial>
-        <origin xyz="4.9801308910080166e-14 0.006389230769241375 -4.5102810375396984e-17" rpy="0 0 0"/>
-        <mass value="0.20037470643677413"/>
-        <inertia ixx="6.9e-05" iyy="0.000135" izz="6.9e-05" ixy="0.0" iyz="0.0" ixz="-0.0"/>
-      </inertial>
-      <visual>
-        <origin xyz="0.005 -0.072 -0.0234" rpy="0 0 0"/>
-        <geometry>
-          <mesh filename="package://faro_description/meshes/wheel_1.stl" scale="0.001 0.001 0.001"/>
-        </geometry>
-        <material name="silver"/>
-      </visual>
-      <collision>
-        <origin xyz="0.005 -0.072 -0.0234" rpy="0 0 0"/>
-        <geometry>
-          <mesh filename="package://faro_description/meshes/wheel_1.stl" scale="0.001 0.001 0.001"/>
-        </geometry>
-      </collision>
-    </link>
+    <inertial>
+      <origin
+        xyz="-2.8093E-09 -1.6256E-09 0.00047467"
+        rpy="0 0 0" />
+      <mass
+        value="0.050589" />
+      <inertia
+        ixx="2.8263E-05"
+        ixy="-1.4586E-12"
+        ixz="1.5929E-12"
+        iyy="2.8263E-05"
+        iyz="1.4235E-12"
+        izz="4.8345E-05" />
+    </inertial>
+    <visual>
+      <origin
+        xyz="0 0 0"
+        rpy="0 0 0" />
+      <geometry>
+        <mesh
+          filename="package://faro_description/meshes/RodaEsquerda_Link.STL" />
+      </geometry>
+      <material
+        name="">
+        <color
+          rgba="1 1 0 1" />
+      </material>
+    </visual>
+    <collision>
+      <origin
+        xyz="0 0 0"
+        rpy="0 0 0" />
+      <geometry>
+        <mesh
+          filename="package://faro_description/meshes/RodaEsquerda_Link.STL" />
+      </geometry>
+    </collision>
+  </link>
   <joint
     name="RodaEsquerda_Joint"
-    type="continuous">
+    type="revolute">
     <origin
       xyz="-0.053091 0.098228 0.011373"
       rpy="1.5708 -0.58968 3.1416" />
     <parent
-      link="Base1_link" />
+      link="base_link" />
     <child
       link="RodaEsquerda_Link" />
     <axis
-      xyz="0 0 0" />
+      xyz="0 0 -1" />
+    <limit
+      lower="-3.14"
+      upper="3.14"
+      effort="0"
+      velocity="0" />
   </joint>
   <link
     name="RodaDireita_Link">
-      <inertial>
-        <origin xyz="4.9791767930962294e-14 -0.006389230769227219 3.469446951953614e-17" rpy="0 0 0"/>
-        <mass value="0.20037470643677413"/>
-        <inertia ixx="6.9e-05" iyy="0.000135" izz="6.9e-05" ixy="-0.0" iyz="-0.0" ixz="0.0"/>
-      </inertial>
-      <visual>
-        <origin xyz="0.005 0.072 -0.0234" rpy="0 0 0"/>
-        <geometry>
-          <mesh filename="package://faro_description/meshes/wheel_2.stl" scale="0.001 0.001 0.001"/>
-        </geometry>
-        <material name="silver"/>
-      </visual>
-      <collision>
-        <origin xyz="0.005 0.072 -0.0234" rpy="0 0 0"/>
-        <geometry>
-          <mesh filename="package://faro_description/meshes/wheel_2.stl" scale="0.001 0.001 0.001"/>
-        </geometry>
-      </collision>
-    </link>
+    <inertial>
+      <origin
+        xyz="0 0 0"
+        rpy="0 0 0" />
+      <mass
+        value="0" />
+      <inertia
+        ixx="0"
+        ixy="0"
+        ixz="0"
+        iyy="0"
+        iyz="0"
+        izz="0" />
+    </inertial>
+    <visual>
+      <origin
+        xyz="0 0 0"
+        rpy="0 0 0" />
+      <geometry>
+        <mesh
+          filename="package://faro_description/meshes/RodaDireita_Link.STL" />
+      </geometry>
+      <material
+        name="">
+        <color
+          rgba="1 1 1 1" />
+      </material>
+    </visual>
+    <collision>
+      <origin
+        xyz="0 0 0"
+        rpy="0 0 0" />
+      <geometry>
+        <mesh
+          filename="package://faro_description/meshes/RodaDireita_Link.STL" />
+      </geometry>
+    </collision>
+  </link>
   <joint
     name="RodaDireita_Joint"
-    type="continuous">
+    type="revolute">
     <origin
       xyz="-0.053091 -0.098296 0.011373"
       rpy="1.5708 -1.1528 0" />
     <parent
-      link="Base1_link" />
+      link="base_link" />
     <child
       link="RodaDireita_Link" />
     <axis
-      xyz="0 0 0" />
-  </joint>
-  <!--<link
-    name="Esfera_Link">
-    <inertial>
-      <origin
-        xyz="0 0 0"
-        rpy="0 0 0" />
-      <mass
-        value="0.010855" />
-      <inertia
-        ixx="2.0829E-07"
-        ixy="-6.6174E-24"
-        ixz="0"
-        iyy="2.0829E-07"
-        iyz="-6.6174E-24"
-        izz="2.0829E-07" />
-    </inertial>
-    <visual>
-      <origin
-        xyz="0 0 0"
-        rpy="0 0 0" />
-      <geometry>
-        <mesh
-          filename="package://faro_description/meshes/Esfera_Link.STL" />
-      </geometry>
-      <material
-        name="">
-        <color
-          rgba="0.89804 0.89804 0.89804 1" />
-      </material>
-    </visual>
-    <collision>
-      <origin
-        xyz="0 0 0"
-        rpy="0 0 0" />
-      <geometry>
-        <mesh
-          filename="package://faro_description/meshes/Esfera_Link.STL" />
-      </geometry>
-    </collision>
-  </link>
-  <joint
-    name="Esfera_Joint"
-    type="continuous">
-    <origin
-      xyz="0 -0.014652 0"
-      rpy="0.50086 -1.1467 -0.05132" />
-    <parent
-      link="Base2_Link" />
-    <child
-      link="Esfera_Link" />
-    <axis
-      xyz="0 0 0" />
+      xyz="0 0 -1" />
     <limit
-      lower="0"
-      upper="0"
+      lower="-3.14"
+      upper="3.14"
       effort="0"
       velocity="0" />
-  </joint>-->
-  <gazebo reference="Base1_link">
+  </joint>
+  <gazebo reference="base_link">
     <material>Gazebo/Green</material>
-  </gazebo>
-  <gazebo reference="RodaEsquerda_Link">
-    <material>Gazebo/Blue</material>
-  </gazebo>
-  <gazebo reference="RodaDireita_Link">
-    <material>Gazebo/Red</material>
   </gazebo>
   <gazebo>
@@ -204,8 +244,8 @@
       <publishTf>1</publishTf>
       <odometryFrame>odom</odometryFrame>
-      <robotBaseFrame>Base1_link</robotBaseFrame>
+      <robotBaseFrame>base_link</robotBaseFrame>
     </plugin>
   </gazebo>
   <!-- Sensor LF -->
-  <xacro:sensor x="0.145" y="0.03" z="0.007" parent="Base1_link"/>
+  <xacro:sensor x="0.145" y="0.03" z="0.007" parent="base_link"/>
 </robot>

Commit message: wheel adjustment

File: urdf/faro.xacro (robot description, xacro)
@@ -3,4 +3,5 @@
   <xacro:include filename="$(find faro_description)/urdf/sensor.xacro"/>
   <xacro:include filename="$(find faro_description)/urdf/common_properties.xacro"/>
+  <xacro:include filename="$(find faro_description)/urdf/wheel.xacro" />
   <!-- Dummy for no warning -->
   <link name="dummy"></link>
@@ -104,123 +105,8 @@
       friction="0" />
   </joint>
-  <link
-    name="RodaEsquerda_Link">
-    <inertial>
-      <origin
-        xyz="-2.8093E-09 -1.6256E-09 0.00047467"
-        rpy="0 0 0" />
-      <mass
-        value="0.050589" />
-      <inertia
-        ixx="2.8263E-05"
-        ixy="-1.4586E-12"
-        ixz="1.5929E-12"
-        iyy="2.8263E-05"
-        iyz="1.4235E-12"
-        izz="4.8345E-05" />
-    </inertial>
-    <visual>
-      <origin
-        xyz="0 0 0"
-        rpy="0 0 0" />
-      <geometry>
-        <mesh
-          filename="package://faro_description/meshes/RodaEsquerda_Link.STL" />
-      </geometry>
-      <material
-        name="">
-        <color
-          rgba="1 1 0 1" />
-      </material>
-    </visual>
-    <collision>
-      <origin
-        xyz="0 0 0"
-        rpy="0 0 0" />
-      <geometry>
-        <mesh
-          filename="package://faro_description/meshes/RodaEsquerda_Link.STL" />
-      </geometry>
-    </collision>
-  </link>
-  <joint
-    name="RodaEsquerda_Joint"
-    type="revolute">
-    <origin
-      xyz="-0.053091 0.098228 0.011373"
-      rpy="1.5708 -0.58968 3.1416" />
-    <parent
-      link="base_link" />
-    <child
-      link="RodaEsquerda_Link" />
-    <axis
-      xyz="0 0 -1" />
-    <limit
-      lower="-3.14"
-      upper="3.14"
-      effort="0"
-      velocity="0" />
-  </joint>
-  <link
-    name="RodaDireita_Link">
-    <inertial>
-      <origin
-        xyz="0 0 0"
-        rpy="0 0 0" />
-      <mass
-        value="0" />
-      <inertia
-        ixx="0"
-        ixy="0"
-        ixz="0"
-        iyy="0"
-        iyz="0"
-        izz="0" />
-    </inertial>
-    <visual>
-      <origin
-        xyz="0 0 0"
-        rpy="0 0 0" />
-      <geometry>
-        <mesh
-          filename="package://faro_description/meshes/RodaDireita_Link.STL" />
-      </geometry>
-      <material
-        name="">
-        <color
-          rgba="1 1 1 1" />
-      </material>
-    </visual>
-    <collision>
-      <origin
-        xyz="0 0 0"
-        rpy="0 0 0" />
-      <geometry>
-        <mesh
-          filename="package://faro_description/meshes/RodaDireita_Link.STL" />
-      </geometry>
-    </collision>
-  </link>
-  <joint
-    name="RodaDireita_Joint"
-    type="revolute">
-    <origin
-      xyz="-0.053091 -0.098296 0.011373"
-      rpy="1.5708 -1.1528 0" />
-    <parent
-      link="base_link" />
-    <child
-      link="RodaDireita_Link" />
-    <axis
-      xyz="0 0 -1" />
-    <limit
-      lower="-3.14"
-      upper="3.14"
-      effort="0"
-      velocity="0" />
-  </joint>
-  <gazebo reference="base_link">
-    <material>Gazebo/Green</material>
-  </gazebo>
+  <!-- Wheels -->
+  <xacro:wheel name="right" position="-0.053091 0.098228 0.011373" stl="RodaDireita_Link.STL" />
+  <xacro:wheel name="left" position="-0.053091 -0.098228 0.011373" stl="RodaEsquerda_Link.STL" />
+  <!-- Pluguins adicionais (NÃO TIRAR) -->
   <gazebo>
     <plugin filename="libgazebo_ros_diff_drive.so" name="differential_drive_controller">
@@ -229,7 +115,7 @@
       <alwaysOn>true</alwaysOn>
       <updateRate>20</updateRate>
-      <leftJoint>RodaEsquerda_Joint</leftJoint>
+      <leftJoint>joint_left_wheel</leftJoint>
       <publishWheelTF>false</publishWheelTF>
-      <rightJoint>RodaDireita_Joint</rightJoint>
+      <rightJoint>joint_right_wheel</rightJoint>
       <wheelSeparation>0.3</wheelSeparation>
       <publishWheelJointState>false</publishWheelJointState>

Commit message: Add files via upload

File: urdf/faro.xacro (robot description, xacro)
@@ -14,15 +14,15 @@
     <inertial>
       <origin
-        xyz="0.00873430427479388 -0.00175292065981603 -1.60683999922646E-05"
-        rpy="0 0 0" />
-      <mass
-        value="0.451148910388453" />
-      <inertia
-        ixx="0.000741612731246182"
-        ixy="1.64659716773886E-06"
-        ixz="1.51707793234015E-07"
-        iyy="0.00220273812328352"
-        iyz="-9.17558592682493E-09"
-        izz="0.00147205616680342" />
+        xyz="0.0174255966476911 0.00801880376211097 0.000514824513657607"
+        rpy="0 0 0" />
+      <mass
+        value="0.571210773201543" />
+      <inertia
+        ixx="0.00106878852176426"
+        ixy="1.64537220733215E-06"
+        ixz="1.51778150035731E-07"
+        iyy="0.00251951460362473"
+        iyz="2.05551196011702E-06"
+        izz="0.00161673123451595" />
     </inertial>
     <visual>
@@ -37,5 +37,5 @@
         name="">
         <color
-          rgba="0.498039215686275 0.498039215686275 0.498039215686275 1" />
+          rgba="0.250980392156863 0.250980392156863 0.250980392156863 1" />
       </material>
     </visual>
@@ -51,18 +51,134 @@
   </link>
   <link
+    name="RodaEsquerda_Link">
+    <inertial>
+      <origin
+        xyz="-2.8092860329676E-09 -1.62563565386797E-09 0.000474666987463443"
+        rpy="0 0 0" />
+      <mass
+        value="0.0505890699400185" />
+      <inertia
+        ixx="2.82629417091323E-05"
+        ixy="-1.45857252989277E-12"
+        ixz="1.5929368350202E-12"
+        iyy="2.82629426261707E-05"
+        iyz="1.42351071240575E-12"
+        izz="4.83451974004371E-05" />
+    </inertial>
+    <visual>
+      <origin
+        xyz="0 0 0"
+        rpy="0 0 0" />
+      <geometry>
+        <mesh
+          filename="package://faro_description/meshes/RodaEsquerda_Link.STL" />
+      </geometry>
+      <material
+        name="">
+        <color
+          rgba="1 1 0 1" />
+      </material>
+    </visual>
+    <collision>
+      <origin
+        xyz="0 0 0"
+        rpy="0 0 0" />
+      <geometry>
+        <mesh
+          filename="package://faro_description/meshes/RodaEsquerda_Link.STL" />
+      </geometry>
+    </collision>
+  </link>
+  <joint
+    name="RodaEsquerda_Joint"
+    type="revolute">
+    <origin
+      xyz="-0.053091 0.098228 0.011373"
+      rpy="1.5708 -0.58968 3.1416" />
+    <parent
+      link="base_link" />
+    <child
+      link="RodaEsquerda_Link" />
+    <axis
+      xyz="0 0 -1" />
+    <limit
+      lower="-3.14"
+      upper="3.14"
+      effort="0"
+      velocity="0" />
+  </joint>
+  <link
+    name="RodaDireita_Link">
+    <inertial>
+      <origin
+        xyz="-1.57279833080948E-09 1.97751798269863E-09 0.000474666390947093"
+        rpy="0 0 0" />
+      <mass
+        value="0.0505890697331487" />
+      <inertia
+        ixx="2.82629424828749E-05"
+        ixy="1.66841255641224E-12"
+        ixz="5.67166595620934E-13"
+        iyy="2.82629415449179E-05"
+        iyz="-1.63581653303395E-12"
+        izz="4.83451973964662E-05" />
+    </inertial>
+    <visual>
+      <origin
+        xyz="0 0 0"
+        rpy="0 0 0" />
+      <geometry>
+        <mesh
+          filename="package://faro_description/meshes/RodaDireita_Link.STL" />
+      </geometry>
+      <material
+        name="">
+        <color
+          rgba="1 1 0 1" />
+      </material>
+    </visual>
+    <collision>
+      <origin
+        xyz="0 0 0"
+        rpy="0 0 0" />
+      <geometry>
+        <mesh
+          filename="package://faro_description/meshes/RodaDireita_Link.STL" />
+      </geometry>
+    </collision>
+  </link>
+  <joint
+    name="RodaDireita_Joint"
+    type="revolute">
+    <origin
+      xyz="-0.053091 -0.098296 0.011373"
+      rpy="1.5708 -1.1528 0" />
+    <parent
+      link="base_link" />
+    <child
+      link="RodaDireita_Link" />
+    <axis
+      xyz="0 0 -1" />
+    <limit
+      lower="-3.14"
+      upper="3.14"
+      effort="0"
+      velocity="0" />
+  </joint>
+  <link
     name="RodaEsferica_Link">
     <inertial>
       <origin
-        xyz="0.068659 -0.017264 0.00018379"
-        rpy="0 0 0" />
-      <mass
-        value="0.020844" />
-      <inertia
-        ixx="9.8497E-07"
-        ixy="1.4029E-22"
-        ixz="-7.8188E-23"
-        iyy="1.4E-06"
-        iyz="1.592E-22"
-        izz="8.9118E-07" />
+        xyz="-5.22644872541084E-05 0.00222455562959233 -0.0010857972628485"
+        rpy="0 0 0" />
+      <mass
+        value="0.020844144758511" />
+      <inertia
+        ixx="9.6931356518338E-07"
+        ixy="7.23987073595594E-09"
+        ixz="3.55631081018164E-08"
+        iyy="1.30556974124119E-06"
+        iyz="-1.93784561089294E-07"
+        izz="1.00125214093605E-06" />
     </inertial>
     <visual>
@@ -77,5 +193,5 @@
         name="">
         <color
-          rgba="0.89804 0.89804 0.89804 1" />
+          rgba="0.898039215686275 0.898039215686275 0.898039215686275 1" />
       </material>
     </visual>
@@ -94,6 +210,6 @@
     type="fixed">
     <origin
-      xyz="0 0 0"
-      rpy="1.5708 0 0" />
+      xyz="0.068659 -0.00018379 -0.01974"
+      rpy="2.0249 0.02111 -2.718" />
     <parent
       link="base_link" />
@@ -104,4 +220,57 @@
     <dynamics
       friction="0" />
+  </joint>
+  <link
+    name="ArUco_Link">
+    <inertial>
+      <origin
+        xyz="-1.38777878078145E-17 0.001 6.93889390390723E-18"
+        rpy="0 0 0" />
+      <mass
+        value="0.0129572802" />
+      <inertia
+        ixx="6.99978201762134E-06"
+        ixy="-4.00894272551875E-40"
+        ixz="-3.10741874939846E-22"
+        iyy="1.39909258484427E-05"
+        iyz="0"
+        izz="6.99978201762134E-06" />
+    </inertial>
+    <visual>
+      <origin
+        xyz="0 0 0"
+        rpy="0 0 0" />
+      <geometry>
+        <mesh
+          filename="package://faro_description/meshes/ArUco_Link.STL" />
+      </geometry>
+      <material
+        name="">
+        <color
+          rgba="0.792156862745098 0.819607843137255 0.933333333333333 1" />
+      </material>
+    </visual>
+    <collision>
+      <origin
+        xyz="0 0 0"
+        rpy="0 0 0" />
+      <geometry>
+        <mesh
+          filename="package://faro_description/meshes/ArUco_Link.STL" />
+      </geometry>
+    </collision>
+  </link>
+  <joint
+    name="ArUco_Joint"
+    type="fixed">
+    <origin
+      xyz="0.050084 -3.3786E-05 0.070373"
+      rpy="1.5708 0 0" />
+    <parent
+      link="base_link" />
+    <child
+      link="ArUco_Link" />
+    <axis
+      xyz="0 0 0" />
   </joint>
   <!-- Wheels -->
